File: hardware/boards/glasgow/io_buffer.sch (KiCad schematic (older format))
At the start: 42 parts, among them J2 Conn_02x10_Odd_Even, U10 DAC081C081CIMK, U11 TPS73101DBV, U16 SN74LVC1T45DRL, U17 SN74LVC1T45DRL, U18 SN74LVC1T45DRL, U19 SN74LVC1T45DRL, U20 SN74LVC1T45DRL, U21 SN74LVC1T45DRL, U5 SN74LVC1T45DRL, U6 SN74LVC1T45DRL, U9 ADC081C021CIMM

Commit message: revC: move FPGA I/O banks to a separate sheet, wire I/O buffers
Parts:
- added RN6: 10K, Resistor_SMD:R_Array_Convex_8x0602, symbol Device:R_Pack08
- added U19: TCA9534, Package_SO:TSSOP-16_4.4x5mm_P0.65mm, symbol Interface_Expansion:TCA9534
Connections:
- net labels added: ADRPULL
- net labels removed: VEXT
- wire segments 193 -> 221
Other:
- note added: "Addr (ADR=L): 0100000\nAddr (ADR=H): 0100001"
- moved on the sheet: U14

Commit message: revC: I/O buffer B routing
Parts:
- removed C29, C34: 4u7, Capacitor_SMD:C_0603_1608Metric_Pad1.05x0.95mm_HandSolder, symbol Device:C
- added C54: u1, Capacitor_SMD:C_0402_1005Metric, symbol Device:C
- added C82, C83: 4u7, Capacitor_SMD:C_0603_1608Metric_Pad1.05x0.95mm_HandSolder, symbol Device:C
- added J6, J7: Conn_01x08, Connector_PinHeader_1.27mm:PinHeader_1x08_P1.27mm_Vertical, symbol Connector_Generic:Conn_01x08
- C39: value 4u7 -> u1; footprint Capacitor_SMD:C_0603_1608Metric_Pad1.05x0.95mm_HandSolder -> Capacitor_SMD:C_0402_1005Metric
Connections:
- wire segments 221 -> 248
Other:
- note added: "ADC/DAC decoupling"
- note removed: "LDO Input Cap"
- moved on the sheet: U14

Commit message: revC: more layout work on port A & misc
Parts:
- added C86, C87: u1, Capacitor_SMD:C_0402_1005Metric, symbol Device:C
- added R38, R39: 10k, Resistor_SMD:R_0402_1005Metric, symbol Device:R
- added U33: TCA9517, Package_SO:VSSOP-8_3.0x3.0mm_P0.65mm, symbol Glasgow:TCA9517
Connections:
- wire segments 248 -> 271

Commit message: revC: I/O buffers fully routed
Parts:
- J6, J7: footprint Connector_PinHeader_1.27mm:PinHeader_1x08_P1.27mm_Vertical -> Connector_PinSocket_1.27mm:PinSocket_1x08_P1.27mm_Vertical

Commit message: revC: use proper footprint for I/O connectors, tweak silkscreen
Parts:
- J2: footprint Connector_PinHeader_2.54mm:PinHeader_2x10_P2.54mm_Vertical -> Connector_IDC:IDC-Header_2x10_P2.54mm_Vertical
Changed lines of the file:
@@
 $Descr A4 11693 8268
 encoding utf-8
-Sheet 4 4
+Sheet 3 4
 Title "I/O Buffer"
 Date ""
@@
 F 0 "J2" H 8300 2100 50  0000 C CNN
 F 1 "Conn_02x10_Odd_Even" H 8300 3226 50  0001 C CNN
-F 2 "Connector_PinHeader_2.54mm:PinHeader_2x10_P2.54mm_Vertical" H 8250 2700 50  0001 C CNN
+F 2 "Connector_IDC:IDC-Header_2x10_P2.54mm_Vertical" H 8250 2700 50  0001 C CNN
 F 3 "https://www.mouser.com/datasheet/2/276/0878342019_PCB_HEADERS-152849.pdf" H 8250 2700 50  0001 C CNN
 F 4 "Molex" H 4550 -450 50  0001 C CNN "Mfg"

Commit message: revC1: add discharge resistors for VIO
Parts:
- added R42: 1k, Resistor_SMD:R_0402_1005Metric, symbol Device:R
Connections:
- wire segments 271 -> 274
Changed lines of the file:
@@
 $Descr A4 11693 8268
 encoding utf-8
-Sheet 3 4
+Sheet 4 4
 Title "I/O Buffer"
 Date ""
@@
 Wire Wire Line
 	6200 2400 7150 2400
+$Comp
+L Device:R R?
+U 1 1 5C5D4477
+P 9600 2000
+AR Path="/5AF7D604/5C5D4477" Ref="R?"  Part="1"
+AR Path="/5AFBDC9E/5C5D4477" Ref="R?"  Part="1"
+AR Path="/5C7B59B0/5C9E337E/5C5D4477" Ref="R42"  Part="1"
+AR Path="/5C7B59B0/5C9E338E/5C5D4477" Ref="R41"  Part="1"
+F 0 "R42" H 9530 1954 50  0000 R CNN
+F 1 "1k" H 9530 2045 50  0000 R CNN
+F 2 "Resistor_SMD:R_0402_1005Metric" V 9530 2000 50  0001 C CNN
+F 3 "https://www.mouser.com/datasheet/2/447/PYu-AC_51_RoHS_L_6-1152827.pdf" H 9600 2000 50  0001 C CNN
+F 4 "Yageo" H 3450 -2950 50  0001 C CNN "Mfg"
+F 5 "RC0603FR-0759KL" H 3450 -2950 50  0001 C CNN "MPN"
+	1    9600 2000
+	-1   0    0    1
+$EndComp
+Wire Wire Line
+	9250 1750 9600 1750
+Wire Wire Line
+	9600 1750 9600 1850
+Connection ~ 9250 1750
+$Comp
+L power:GND #PWR?
+U 1 1 5C5E94B2
+P 9600 2200
+AR Path="/5AF7D604/5C5E94B2" Ref="#PWR?"  Part="1"
+AR Path="/5AFBDC9E/5C5E94B2" Ref="#PWR?"  Part="1"
+AR Path="/5C7B59B0/5C9E337E/5C5E94B2" Ref="#PWR0133"  Part="1"
+AR Path="/5C7B59B0/5C9E338E/5C5E94B2" Ref="#PWR0131"  Part="1"
+F 0 "#PWR0133" H 9600 1950 50  0001 C CNN
+F 1 "GND" H 9605 2027 50  0000 C CNN
+F 2 "" H 9600 2200 50  0001 C CNN
+F 3 "" H 9600 2200 50  0001 C CNN
+	1    9600 2200
+	1    0    0    -1
+$EndComp
+Wire Wire Line
+	9600 2150 9600 2200
 $EndSCHEMATC
