File: hardware/boards/test-jig/led-board.sch (KiCad schematic (older format))
At the start: 26 parts, among them J6 Conn_02x05_Odd_Even

Commit message: test-jig: assign footprints (except terminals to pogo pins)
Parts:
- C13: footprint (none) -> Capacitor_SMD:C_0603_1608Metric_Pad1.05x0.95mm_HandSolder
- D10, D11, D2, D3, D4, D5, D6, D7, D8, D9: footprint (none) -> LED_SMD:LED_0603_1608Metric_Castellated
- H5, H6, H7, H8: footprint (none) -> MountingHole:MountingHole_3.7mm_Pad_Via
- J6: footprint (none) -> Connector_IDC:IDC-Header_2x05_P2.54mm_Vertical
- R26, R27, R28, R29, R30, R31, R32, R33, R34, R35: footprint (none) -> Resistor_SMD:R_0603_1608Metric_Pad1.05x0.95mm_HandSolder
Changed lines of the file:
@@
 F 0 "D2" H 5293 2395 50  0000 C CNN
 F 1 "green" H 5293 2486 50  0000 C CNN
-F 2 "" H 5300 2650 50  0001 C CNN
+F 2 "LED_SMD:LED_0603_1608Metric_Castellated" H 5300 2650 50  0001 C CNN
 F 3 "~" H 5300 2650 50  0001 C CNN
 	1    5300 2650
@@
 F 0 "R26" V 4643 2650 50  0000 C CNN
 F 1 "2k2" V 4734 2650 50  0000 C CNN
-F 2 "" V 4780 2650 50  0001 C CNN
+F 2 "Resistor_SMD:R_0603_1608Metric_Pad1.05x0.95mm_HandSolder" V 4780 2650 50  0001 C CNN
 F 3 "~" H 4850 2650 50  0001 C CNN
 	1    4850 2650
@@
 F 0 "J6" V 2300 4512 50  0000 R CNN
 F 1 "Conn_02x05_Odd_Even" V 2255 4512 50  0001 R CNN
-F 2 "" H 2250 4800 50  0001 C CNN
+F 2 "Connector_IDC:IDC-Header_2x05_P2.54mm_Vertical" H 2250 4800 50  0001 C CNN
 F 3 "~" H 2250 4800 50  0001 C CNN
 	1    2250 4800
@@
 F 0 "D4" H 5293 3295 50  0000 C CNN
 F 1 "red" H 5293 3386 50  0000 C CNN
-F 2 "" H 5300 3550 50  0001 C CNN
+F 2 "LED_SMD:LED_0603_1608Metric_Castellated" H 5300 3550 50  0001 C CNN
 F 3 "~" H 5300 3550 50  0001 C CNN
 	1    5300 3550
@@
 F 0 "D3" H 3643 3295 50  0000 C CNN
 F 1 "green" H 3643 3386 50  0000 C CNN
-F 2 "" H 3650 3550 50  0001 C CNN
+F 2 "LED_SMD:LED_0603_1608Metric_Castellated" H 3650 3550 50  0001 C CNN
 F 3 "~" H 3650 3550 50  0001 C CNN
 	1    3650 3550
@@
 F 0 "R27" V 3893 3550 50  0000 C CNN
 F 1 "2k2" V 3984 3550 50  0000 C CNN
-F 2 "" V 4030 3550 50  0001 C CNN
+F 2 "Resistor_SMD:R_0603_1608Metric_Pad1.05x0.95mm_HandSolder" V 4030 3550 50  0001 C CNN
 F 3 "~" H 4100 3550 50  0001 C CNN
 	1    4100 3550
@@
 F 0 "R28" V 4643 3550 50  0000 C CNN
 F 1 "2k2" V 4734 3550 50  0000 C CNN
-F 2 "" V 4780 3550 50  0001 C CNN
+F 2 "Resistor_SMD:R_0603_1608Metric_Pad1.05x0.95mm_HandSolder" V 4780 3550 50  0001 C CNN
 F 3 "~" H 4850 3550 50  0001 C CNN
 	1    4850 3550
@@
 F 0 "D7" H 5293 3995 50  0000 C CNN
 F 1 "red" H 5293 4086 50  0000 C CNN
-F 2 "" H 5300 4250 50  0001 C CNN
+F 2 "LED_SMD:LED_0603_1608Metric_Castellated" H 5300 4250 50  0001 C CNN
 F 3 "~" H 5300 4250 50  0001 C CNN
 	1    5300 4250
@@
 F 0 "D6" H 3643 3995 50  0000 C CNN
 F 1 "green" H 3643 4086 50  0000 C CNN
-F 2 "" H 3650 4250 50  0001 C CNN
+F 2 "LED_SMD:LED_0603_1608Metric_Castellated" H 3650 4250 50  0001 C CNN
 F 3 "~" H 3650 4250 50  0001 C CNN
 	1    3650 4250
@@
 F 0 "R30" V 3893 4250 50  0000 C CNN
 F 1 "2k2" V 3984 4250 50  0000 C CNN
-F 2 "" V 4030 4250 50  0001 C CNN
+F 2 "Resistor_SMD:R_0603_1608Metric_Pad1.05x0.95mm_HandSolder" V 4030 4250 50  0001 C CNN
 F 3 "~" H 4100 4250 50  0001 C CNN
 	1    4100 4250
@@
 F 0 "R31" V 4643 4250 50  0000 C CNN
 F 1 "2k2" V 4734 4250 50  0000 C CNN
-F 2 "" V 4780 4250 50  0001 C CNN
+F 2 "Resistor_SMD:R_0603_1608Metric_Pad1.05x0.95mm_HandSolder" V 4780 4250 50  0001 C CNN
 F 3 "~" H 4850 4250 50  0001 C CNN
 	1    4850 4250
@@
 F 0 "D11" H 5293 4745 50  0000 C CNN
 F 1 "red" H 5293 4836 50  0000 C CNN
-F 2 "" H 5300 5000 50  0001 C CNN
+F 2 "LED_SMD:LED_0603_1608Metric_Castellated" H 5300 5000 50  0001 C CNN
 F 3 "~" H 5300 5000 50  0001 C CNN
 	1    5300 5000
@@
 F 0 "D10" H 3643 4745 50  0000 C CNN
 F 1 "green" H 3643 4836 50  0000 C CNN
-F 2 "" H 3650 5000 50  0001 C CNN
+F 2 "LED_SMD:LED_0603_1608Metric_Castellated" H 3650 5000 50  0001 C CNN
 F 3 "~" H 3650 5000 50  0001 C CNN
 	1    3650 5000
@@
 F 0 "R34" V 3893 5000 50  0000 C CNN
 F 1 "2k2" V 3984 5000 50  0000 C CNN
-F 2 "" V 4030 5000 50  0001 C CNN
+F 2 "Resistor_SMD:R_0603_1608Metric_Pad1.05x0.95mm_HandSolder" V 4030 5000 50  0001 C CNN
 F 3 "~" H 4100 5000 50  0001 C CNN
 	1    4100 5000
@@
 F 0 "R35" V 4643 5000 50  0000 C CNN
 F 1 "2k2" V 4734 5000 50  0000 C CNN
-F 2 "" V 4780 5000 50  0001 C CNN
+F 2 "Resistor_SMD:R_0603_1608Metric_Pad1.05x0.95mm_HandSolder" V 4780 5000 50  0001 C CNN
 F 3 "~" H 4850 5000 50  0001 C CNN
 	1    4850 5000
@@
 F 0 "C13" H 2915 4796 50  0000 L CNN
 F 1 "100nF" H 2915 4705 50  0000 L CNN
-F 2 "" H 2838 4600 50  0001 C CNN
+F 2 "Capacitor_SMD:C_0603_1608Metric_Pad1.05x0.95mm_HandSolder" H 2838 4600 50  0001 C CNN
 F 3 "~" H 2800 4750 50  0001 C CNN
 	1    2800 4750
@@
 F 0 "D5" H 8293 3545 50  0000 C CNN
 F 1 "yellow" H 8293 3636 50  0000 C CNN
-F 2 "" H 8300 3800 50  0001 C CNN
+F 2 "LED_SMD:LED_0603_1608Metric_Castellated" H 8300 3800 50  0001 C CNN
 F 3 "~" H 8300 3800 50  0001 C CNN
 	1    8300 3800
@@
 F 0 "D8" H 8293 3995 50  0000 C CNN
 F 1 "green" H 8293 4086 50  0000 C CNN
-F 2 "" H 8300 4250 50  0001 C CNN
+F 2 "LED_SMD:LED_0603_1608Metric_Castellated" H 8300 4250 50  0001 C CNN
 F 3 "~" H 8300 4250 50  0001 C CNN
 	1    8300 4250
@@
 F 0 "D9" H 8293 4445 50  0000 C CNN
 F 1 "red" H 8293 4536 50  0000 C CNN
-F 2 "" H 8300 4700 50  0001 C CNN
+F 2 "LED_SMD:LED_0603_1608Metric_Castellated" H 8300 4700 50  0001 C CNN
 F 3 "~" H 8300 4700 50  0001 C CNN
 	1    8300 4700
@@
 F 0 "R29" V 7643 3800 50  0000 C CNN
 F 1 "2k2" V 7734 3800 50  0000 C CNN
-F 2 "" V 7780 3800 50  0001 C CNN
+F 2 "Resistor_SMD:R_0603_1608Metric_Pad1.05x0.95mm_HandSolder" V 7780 3800 50  0001 C CNN
 F 3 "~" H 7850 3800 50  0001 C CNN
 	1    7850 3800
@@
 F 0 "R32" V 7643 4250 50  0000 C CNN
 F 1 "2k2" V 7734 4250 50  0000 C CNN
-F 2 "" V 7780 4250 50  0001 C CNN
+F 2 "Resistor_SMD:R_0603_1608Metric_Pad1.05x0.95mm_HandSolder" V 7780 4250 50  0001 C CNN
 F 3 "~" H 7850 4250 50  0001 C CNN
 	1    7850 4250
@@
 F 0 "R33" V 7643 4700 50  0000 C CNN
 F 1 "2k2" V 7734 4700 50  0000 C CNN
-F 2 "" V 7780 4700 50  0001 C CNN
+F 2 "Resistor_SMD:R_0603_1608Metric_Pad1.05x0.95mm_HandSolder" V 7780 4700 50  0001 C CNN
 F 3 "~" H 7850 4700 50  0001 C CNN
 	1    7850 4700
@@
 F 0 "H5" H 2650 6653 50  0000 L CNN
 F 1 "MountingHole_Pad" H 2650 6608 50  0001 L CNN
-F 2 "" H 2550 6650 50  0001 C CNN
+F 2 "MountingHole:MountingHole_3.7mm_Pad_Via" H 2550 6650 50  0001 C CNN
 F 3 "~" H 2550 6650 50  0001 C CNN
 	1    2550 6650
@@
 F 0 "H6" H 2950 6653 50  0000 L CNN
 F 1 "MountingHole_Pad" H 2950 6608 50  0001 L CNN
-F 2 "" H 2850 6650 50  0001 C CNN
+F 2 "MountingHole:MountingHole_3.7mm_Pad_Via" H 2850 6650 50  0001 C CNN
 F 3 "~" H 2850 6650 50  0001 C CNN
 	1    2850 6650
@@
 F 0 "H7" H 3250 6653 50  0000 L CNN
 F 1 "MountingHole_Pad" H 3250 6608 50  0001 L CNN
-F 2 "" H 3150 6650 50  0001 C CNN
+F 2 "MountingHole:MountingHole_3.7mm_Pad_Via" H 3150 6650 50  0001 C CNN
 F 3 "~" H 3150 6650 50  0001 C CNN
 	1    3150 6650
@@
 F 0 "H8" H 3550 6653 50  0000 L CNN
 F 1 "MountingHole_Pad" H 3550 6608 50  0001 L CNN
-F 2 "" H 3450 6650 50  0001 C CNN
+F 2 "MountingHole:MountingHole_3.7mm_Pad_Via" H 3450 6650 50  0001 C CNN
 F 3 "~" H 3450 6650 50  0001 C CNN
 	1    3450 6650
