File: hardware/boards/glasgow/revD1/fpga.kicad_sch (KiCad schematic)
At the start: 57 parts, among them J4 SYNC, J5 JTAG, U10 74AXP1T45, U74 74AXP1T45, U8 LFE5U-25F-8BG256x, U9 W25Q32JVZP

Commit message: hardware: revD1: change MPN of U9 to W25Q32JVZPIM.
Winbond W25Q32JVZPIQ has QE fixed to 1 and nHOLD disabled, which will
break bitstream loading via the FX2. The -IM variant is different only
in that QE is not fixed and defaults to 0.
Parts:
- U9: MPN W25Q32JVZPIQ -> W25Q32JVZPIM
Changed lines of the file:
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@@
 			)
 		)
-		(property "MPN" "W25Q32JVZPIQ"
+		(property "MPN" "W25Q32JVZPIM"
 			(at 60.96 132.08 0)
 			(hide yes)
